File: robotron 057-8606.kicad_pcb (KiCad board)
At the start: 2 copper layers, 20 parts, among them U1 74LS193, U10 74LS123, U11 74LS193, U12 SN75107, U13 SN75110, U15 SN75110, U16 SN75110, U17 SN75110, U18 SN75110, U19 SN75110, U2 74LS193, U3 74LS193, U4 74LS193, U5 74LS193, U9 SN75107, X1 EFS29

Commit message: Einige Verbindungen im Bereich des Zählers ermittelt
Parts:
- added J5: Conn_02x13_Odd_Even, Connector_IDC:IDC-Header_2x13_P2.54mm_Latch6.5mm_Vertical, F.Cu at (6.83, 132.6)
- added R1: R, Resistor_THT:R_Axial_DIN0207_L6.3mm_D2.5mm_P7.62mm_Horizontal, F.Cu at (186.7, 16.8)
- added R2: R, Resistor_THT:R_Axial_DIN0207_L6.3mm_D2.5mm_P7.62mm_Horizontal, F.Cu at (187.5, 21.8)
- added R3: 4,7KΩ, Resistor_THT:R_Axial_DIN0207_L6.3mm_D2.5mm_P7.62mm_Horizontal, F.Cu at (143.0, 40.3)
- added R5: R, Resistor_THT:R_Axial_DIN0207_L6.3mm_D2.5mm_P7.62mm_Horizontal, F.Cu at (80.8, 51.8)
- added U14: 74LS30, Package_DIP:DIP-14_W7.62mm, F.Cu at (202.9, 128.8)
- added U6: 74LS04, Package_DIP:DIP-14_W7.62mm, F.Cu at (241.7, 98.7)
- added U7: 74LS00, Package_DIP:DIP-14_W7.62mm, F.Cu at (217.9, 98.4)
- added U8: 74LS08, Package_DIP:DIP-14_W7.62mm, F.Cu at (202.9, 98.6)
- added X2: EFS13 Interleaved, Connector_IDC:IDC-Header_2x13_P2.54mm_Vertical, F.Cu at (256.7, 112.5)
- added X3: EFS13, Connector_IDC:IDC-Header_2x13_P2.54mm_Vertical, F.Cu at (134.6, 70.7)
- added X4: Conn_02x30_Top_Bottom, Connector_PinHeader_2.54mm:PinHeader_2x30_P2.54mm_Horizontal, F.Cu at (78.9, 153.3)
- moved R6 102.6 mm to (150.5, 51.7), turned to 180 degrees
- moved R4 92.5 mm to (150.6, 45.6), turned to 180 degrees
- moved U10 0.22 mm to (166.6, 101.2)
Connections:
- U1 pad 1: unconnected-(U1-B-Pad1) -> Net-(U1-A)
- U1 pad 10: unconnected-(U1-C-Pad10) -> Net-(U1-A)
- U1 pad 11: unconnected-(U1-~{LOAD}-Pad11) -> Net-(U1-~{LOAD})
- U1 pad 14: unconnected-(U1-CLR-Pad14) -> Net-(U1-A)
- U1 pad 15: unconnected-(U1-A-Pad15) -> Net-(U1-A)
- U1 pad 16: unconnected-(U1-VCC-Pad16) -> +5V
- U1 pad 4: unconnected-(U1-DOWN-Pad4) -> Net-(U1-DOWN)
- U1 pad 5: unconnected-(U1-UP-Pad5) -> /Counter/CLK_UP
- U1 pad 7: unconnected-(U1-QD-Pad7) -> Net-(U1-QD)
- U1 pad 8: unconnected-(U1-GND-Pad8) -> GND
- U1 pad 9: unconnected-(U1-D-Pad9) -> Net-(U1-A)
- U10 pad 4: unconnected-(U10A-~{Q}-Pad4) -> Net-(U10A-~{Q})
- U11 pad 1: unconnected-(U11-B-Pad1) -> GND
- U11 pad 10: unconnected-(U11-C-Pad10) -> GND
- U11 pad 11: unconnected-(U11-~{LOAD}-Pad11) -> Net-(U1-~{LOAD})
- U11 pad 14: unconnected-(U11-CLR-Pad14) -> GND
- U11 pad 15: unconnected-(U11-A-Pad15) -> /Counter/CLK_UP
- U11 pad 16: unconnected-(U11-VCC-Pad16) -> +5V
- U11 pad 4: unconnected-(U11-DOWN-Pad4) -> Net-(U11-DOWN)
- U11 pad 5: unconnected-(U11-UP-Pad5) -> /Counter/CLK_UP
- U11 pad 8: unconnected-(U11-GND-Pad8) -> GND
- U11 pad 9: unconnected-(U11-D-Pad9) -> GND
- U2 pad 1: unconnected-(U2-B-Pad1) -> Net-(U2-B)
- U2 pad 10: unconnected-(U2-C-Pad10) -> GND
- U2 pad 11: unconnected-(U2-~{LOAD}-Pad11) -> Net-(U1-~{LOAD})
- U2 pad 13: unconnected-(U2-~{BO}-Pad13) -> Net-(U2-~{BO})
- U2 pad 14: unconnected-(U2-CLR-Pad14) -> GND
- U2 pad 16: unconnected-(U2-VCC-Pad16) -> +5V
- U2 pad 4: unconnected-(U2-DOWN-Pad4) -> Net-(U1-QD)
- U2 pad 5: unconnected-(U2-UP-Pad5) -> /Counter/CLK_UP
- U2 pad 8: unconnected-(U2-GND-Pad8) -> GND
- U2 pad 9: unconnected-(U2-D-Pad9) -> Net-(U2-A)
- U3 pad 10: unconnected-(U3-C-Pad10) -> Net-(U3-C)
- U3 pad 11: unconnected-(U3-~{LOAD}-Pad11) -> Net-(U1-~{LOAD})
- U3 pad 14: unconnected-(U3-CLR-Pad14) -> GND
- U3 pad 16: unconnected-(U3-VCC-Pad16) -> +5V
- U3 pad 4: unconnected-(U3-DOWN-Pad4) -> Net-(U2-~{BO})
- U3 pad 5: unconnected-(U3-UP-Pad5) -> /Counter/CLK_UP
- U3 pad 8: unconnected-(U3-GND-Pad8) -> GND
- U3 pad 9: unconnected-(U3-D-Pad9) -> GND
- U4 pad 11: unconnected-(U4-~{LOAD}-Pad11) -> Net-(U4-~{LOAD})
- U4 pad 14: unconnected-(U4-CLR-Pad14) -> GND
- U4 pad 16: unconnected-(U4-VCC-Pad16) -> +5V
- U4 pad 4: unconnected-(U4-DOWN-Pad4) -> Net-(U10A-~{Q})
- U4 pad 5: unconnected-(U4-UP-Pad5) -> /Counter/CLK_UP
- U4 pad 8: unconnected-(U4-GND-Pad8) -> GND
- U5 pad 1: unconnected-(U5-B-Pad1) -> /Counter/CLK_UP
- U5 pad 10: unconnected-(U5-C-Pad10) -> /Counter/CLK_UP
- U5 pad 11: unconnected-(U5-~{LOAD}-Pad11) -> Net-(U4-~{LOAD})
- U5 pad 13: unconnected-(U5-~{BO}-Pad13) -> Net-(U11-DOWN)
- U5 pad 14: unconnected-(U5-CLR-Pad14) -> GND
- U5 pad 15: unconnected-(U5-A-Pad15) -> /Counter/CLK_UP
- U5 pad 16: unconnected-(U5-VCC-Pad16) -> +5V
- U5 pad 5: unconnected-(U5-UP-Pad5) -> /Counter/CLK_UP
- U5 pad 8: unconnected-(U5-GND-Pad8) -> GND
- U5 pad 9: unconnected-(U5-D-Pad9) -> /Counter/CLK_UP

Commit message: Aufnahme Schaltplan wip
Parts:
- added R10: 470Ω, Resistor_THT:R_Axial_DIN0207_L6.3mm_D2.5mm_P7.62mm_Horizontal, F.Cu at (142.7, 70.7)
- added R11: R, Resistor_THT:R_Axial_DIN0207_L6.3mm_D2.5mm_P7.62mm_Horizontal, F.Cu at (59.6, 72.4)
- added R7: 4,7KΩ, Resistor_THT:R_Axial_DIN0207_L6.3mm_D2.5mm_P7.62mm_Horizontal, F.Cu at (142.9, 53.1)
- added R8: 470Ω, Resistor_THT:R_Axial_DIN0207_L6.3mm_D2.5mm_P7.62mm_Horizontal, F.Cu at (59.7, 61.2)
- added R9: 470Ω, Resistor_THT:R_Axial_DIN0207_L6.3mm_D2.5mm_P7.62mm_Horizontal, F.Cu at (142.6, 66.9)
- added RN10: 68Ω, Resistor_THT:R_Array_SIP6, F.Cu at (98.9, 113.7)
- added RN11: 68Ω, Resistor_THT:R_Array_SIP6, F.Cu at (94.6, 113.7)
- added RN2: 68Ω, Resistor_THT:R_Array_SIP6, F.Cu at (117.3, 46.7)
- added RN3: 68Ω, Resistor_THT:R_Array_SIP6, F.Cu at (72.3, 65.2)
- added RN5: 68Ω, Resistor_THT:R_Array_SIP6, F.Cu at (222.6, 134.0)
- added RN6: 68Ω, Resistor_THT:R_Array_SIP6, F.Cu at (175.0, 113.4)
- added RN7: 68Ω, Resistor_THT:R_Array_SIP6, F.Cu at (153.9, 113.9)
- added RN8: 68Ω, Resistor_THT:R_Array_SIP6, F.Cu at (136.5, 113.2)
- added RN9: 68Ω, Resistor_THT:R_Array_SIP6, F.Cu at (118.6, 115.8)
- R1, R5: value R -> 470Ω
- R2: value R -> 22Ω
- moved RN1 155.7 mm to (122.2, 46.6), turned to -90 degrees
- moved R6 2.41 mm to (150.5, 49.3)
- moved X2 0.77 mm to (256.5, 113.3)
- moved R4 0.25 mm to (150.6, 45.3)

Commit message: weitere verdrahtungen nachvollzogen
Parts:
- added C1: C_Small, Capacitor_THT:C_Disc_D3.0mm_W1.6mm_P2.50mm, F.Cu at (200.4, 20.8)
- added C10: C_Small, Capacitor_THT:C_Disc_D3.0mm_W1.6mm_P2.50mm, F.Cu at (115.3, 185.9)
- added C11: C_Small, Capacitor_THT:C_Disc_D3.0mm_W1.6mm_P2.50mm, F.Cu at (120.9, 167.0)
- added C12: C_Small, Capacitor_THT:C_Disc_D3.0mm_W1.6mm_P2.50mm, F.Cu at (120.9, 170.2)
- added C13: C_Small, Capacitor_THT:C_Disc_D3.0mm_W1.6mm_P2.50mm, F.Cu at (120.9, 173.3)
- added C14: C_Small, Capacitor_THT:C_Disc_D3.0mm_W1.6mm_P2.50mm, F.Cu at (120.9, 176.5)
- added C15: C_Small, Capacitor_THT:C_Disc_D3.0mm_W1.6mm_P2.50mm, F.Cu at (120.9, 179.6)
- added C16: C_Small, Capacitor_THT:C_Disc_D3.0mm_W1.6mm_P2.50mm, F.Cu at (120.9, 182.8)
- added C17: C_Small, Capacitor_THT:C_Disc_D3.0mm_W1.6mm_P2.50mm, F.Cu at (120.9, 185.9)
- added C2: C_Small, Capacitor_THT:C_Disc_D3.0mm_W1.6mm_P2.50mm, F.Cu at (115.3, 167.0)
- added C3: C_Small, Capacitor_THT:C_Disc_D3.0mm_W1.6mm_P2.50mm, F.Cu at (115.3, 170.2)
- added C4: C_Small, Capacitor_THT:C_Disc_D3.0mm_W1.6mm_P2.50mm, F.Cu at (115.3, 173.3)
- added C5: C_Small, Capacitor_THT:C_Disc_D3.0mm_W1.6mm_P2.50mm, F.Cu at (115.3, 176.5)
- added C6: C_Small, Capacitor_THT:C_Disc_D3.0mm_W1.6mm_P2.50mm, F.Cu at (115.3, 179.6)
- added C7: C_Small, Capacitor_THT:C_Disc_D3.0mm_W1.6mm_P2.50mm, F.Cu at (115.3, 182.8)
- added C8: C_Small, Capacitor_THT:C_Disc_D3.0mm_W1.6mm_P2.50mm, F.Cu at (171.2, 86.1)
- added C9: C_Small, Capacitor_THT:C_Disc_D3.0mm_W1.6mm_P2.50mm, F.Cu at (156.0, 98.8)
- added R12: R, Resistor_THT:R_Axial_DIN0207_L6.3mm_D2.5mm_P7.62mm_Horizontal, F.Cu at (59.4, 75.5)
- added R13: R, Resistor_THT:R_Axial_DIN0207_L6.3mm_D2.5mm_P7.62mm_Horizontal, F.Cu at (119.6, 83.8)
- added R14: R, Resistor_THT:R_Axial_DIN0207_L6.3mm_D2.5mm_P7.62mm_Horizontal, F.Cu at (59.4, 78.5)
- added R15: R, Resistor_THT:R_Axial_DIN0207_L6.3mm_D2.5mm_P7.62mm_Horizontal, F.Cu at (59.4, 81.5)
- added R16: R, Resistor_THT:R_Axial_DIN0207_L6.3mm_D2.5mm_P7.62mm_Horizontal, F.Cu at (59.3, 84.5)
- added R17: R, Resistor_THT:R_Axial_DIN0207_L6.3mm_D2.5mm_P7.62mm_Horizontal, F.Cu at (59.3, 87.4)
- added R18: R, Resistor_THT:R_Axial_DIN0207_L6.3mm_D2.5mm_P7.62mm_Horizontal, F.Cu at (126.7, 80.4)
- added R19: R, Resistor_THT:R_Axial_DIN0207_L6.3mm_D2.5mm_P7.62mm_Horizontal, F.Cu at (126.7, 84.5)
- added R20: R, Resistor_THT:R_Axial_DIN0207_L6.3mm_D2.5mm_P7.62mm_Horizontal, F.Cu at (126.7, 88.5)
- added R21: R, Resistor_THT:R_Axial_DIN0207_L6.3mm_D2.5mm_P7.62mm_Horizontal, F.Cu at (126.7, 92.1)
- added R22: R, Resistor_THT:R_Axial_DIN0207_L6.3mm_D2.5mm_P7.62mm_Horizontal, F.Cu at (172.0, 101.2)
- added R23: R, Resistor_THT:R_Axial_DIN0207_L6.3mm_D2.5mm_P7.62mm_Horizontal, F.Cu at (153.3, 101.3)
- added R24: R, Resistor_THT:R_Axial_DIN0207_L6.3mm_D2.5mm_P7.62mm_Horizontal, F.Cu at (59.2, 90.7)
- added R25: R, Resistor_THT:R_Axial_DIN0207_L6.3mm_D2.5mm_P7.62mm_Horizontal, F.Cu at (59.2, 94.8)
- added R26: R, Resistor_THT:R_Axial_DIN0207_L6.3mm_D2.5mm_P7.62mm_Horizontal, F.Cu at (59.2, 98.8)
- added R27: R, Resistor_THT:R_Axial_DIN0207_L6.3mm_D2.5mm_P7.62mm_Horizontal, F.Cu at (59.2, 102.9)
- added R28: R, Resistor_THT:R_Axial_DIN0207_L6.3mm_D2.5mm_P7.62mm_Horizontal, F.Cu at (59.2, 106.9)
- added R29: R, Resistor_THT:R_Axial_DIN0207_L6.3mm_D2.5mm_P7.62mm_Horizontal, F.Cu at (246.6, 134.9)
- added R30: R, Resistor_THT:R_Axial_DIN0207_L6.3mm_D2.5mm_P7.62mm_Horizontal, F.Cu at (246.6, 138.9)
- added R31: R, Resistor_THT:R_Axial_DIN0207_L6.3mm_D2.5mm_P7.62mm_Horizontal, F.Cu at (233.9, 134.9)
- added R32: R, Resistor_THT:R_Axial_DIN0207_L6.3mm_D2.5mm_P7.62mm_Horizontal, F.Cu at (233.9, 138.9)
- added RN12: 68Ω, Resistor_THT:R_Array_SIP6, F.Cu at (74.4, 75.6)
- R5, R8: value 470Ω -> R
- R7: value 4,7KΩ -> R
- moved R10 0.28 mm to (142.5, 70.9)
- moved R9 0.18 mm to (142.5, 66.8)
Connections:
- net /Driver/UNIT-SELECT renamed /UNIT-SELECT-X5
- net /Driver//UNIT-SELECT renamed //UNIT-SELECT-X5
- R10 pad 2: unconnected-(R10-Pad2) -> Net-(U9-2B)
- R9 pad 2: unconnected-(R9-Pad2) -> Net-(U9-2A)
- RN10 pad 5: unconnected-(RN10-R3-Pad5) -> Net-(RN10-R3)
- RN10 pad 6: unconnected-(RN10-R4-Pad6) -> Net-(RN10-R4)
- RN5 pad 1: unconnected-(RN5-common-Pad1) -> GND
- RN5 pad 2: unconnected-(RN5-R1-Pad2) -> Net-(RN5-R1)
- RN5 pad 3: unconnected-(RN5-R2-Pad3) -> Net-(RN5-R2)
- RN5 pad 5: unconnected-(RN5-R3-Pad5) -> Net-(RN5-R3)
- RN5 pad 6: unconnected-(RN5-R4-Pad6) -> Net-(RN5-R4)
- RN6 pad 1: unconnected-(RN6-common-Pad1) -> GND
- RN6 pad 2: unconnected-(RN6-R1-Pad2) -> Net-(RN6-R1)
- RN6 pad 3: unconnected-(RN6-R2-Pad3) -> Net-(RN6-R2)
- RN6 pad 5: unconnected-(RN6-R3-Pad5) -> Net-(RN6-R3)
- RN6 pad 6: unconnected-(RN6-R4-Pad6) -> Net-(RN6-R4)
- RN7 pad 1: unconnected-(RN7-common-Pad1) -> GND
- RN7 pad 2: unconnected-(RN7-R1-Pad2) -> Net-(RN7-R1)
- RN7 pad 3: unconnected-(RN7-R2-Pad3) -> Net-(RN7-R2)
- RN7 pad 5: unconnected-(RN7-R3-Pad5) -> Net-(RN7-R3)
- RN7 pad 6: unconnected-(RN7-R4-Pad6) -> Net-(RN7-R4)
- RN8 pad 1: unconnected-(RN8-common-Pad1) -> GND
- RN8 pad 2: unconnected-(RN8-R1-Pad2) -> Net-(RN8-R1)
- RN8 pad 3: unconnected-(RN8-R2-Pad3) -> Net-(RN8-R2)
- RN8 pad 5: unconnected-(RN8-R3-Pad5) -> Net-(RN8-R3)
- RN8 pad 6: unconnected-(RN8-R4-Pad6) -> Net-(RN8-R4)
- RN9 pad 1: unconnected-(RN9-common-Pad1) -> GND
- RN9 pad 2: unconnected-(RN9-R1-Pad2) -> Net-(RN9-R1)
- RN9 pad 3: unconnected-(RN9-R2-Pad3) -> Net-(RN9-R2)
- RN9 pad 5: unconnected-(RN9-R3-Pad5) -> Net-(RN9-R3)
- RN9 pad 6: unconnected-(RN9-R4-Pad6) -> Net-(RN9-R4)
- U10 pad 1: unconnected-(U10A-A-Pad1) -> Net-(U10A-A)
- U10 pad 10: unconnected-(U10B-B-Pad10) -> /Counter/CLK_UP
- U10 pad 11: unconnected-(U10B-Clr-Pad11) -> /Counter/CLK_UP
- U10 pad 13: unconnected-(U10A-Q-Pad13) -> /Counter/MonoflopA
- U10 pad 14: unconnected-(U10A-Cext-Pad14) -> Net-(U10A-Cext)
- U10 pad 15: unconnected-(U10A-RCext-Pad15) -> Net-(U10A-RCext)
- U10 pad 2: unconnected-(U10A-B-Pad2) -> /Counter/CLK_UP
- U10 pad 3: unconnected-(U10A-Clr-Pad3) -> /Counter/CLK_UP
- U10 pad 6: unconnected-(U10B-Cext-Pad6) -> Net-(U10B-Cext)
- U10 pad 7: unconnected-(U10B-RCext-Pad7) -> Net-(U10B-RCext)
- U10 pad 9: unconnected-(U10B-A-Pad9) -> Net-(U10A-A)
- U12 pad 4: unconnected-(U12-1Y-Pad4) -> /Counter/UNIT_SELECT_TTL
- U13 pad 1: unconnected-(U13-1A-Pad1) -> Net-(U13-1A)
- U13 pad 10: unconnected-(U13-D-Pad10) -> Net-(U13-1C)
- U13 pad 12: unconnected-(U13-1Z-Pad12) -> Net-(RN5-R1)
- U13 pad 13: unconnected-(U13-1Y-Pad13) -> Net-(RN5-R2)
- U13 pad 2: unconnected-(U13-1B-Pad2) -> Net-(U13-1A)
- U13 pad 3: unconnected-(U13-1C-Pad3) -> Net-(U13-1C)
- U13 pad 4: unconnected-(U13-2C-Pad4) -> Net-(U13-1C)
- U13 pad 5: unconnected-(U13-2A-Pad5) -> Net-(U13-2A)
- U13 pad 6: unconnected-(U13-2B-Pad6) -> Net-(U13-2A)
- U13 pad 8: unconnected-(U13-2Y-Pad8) -> Net-(RN5-R4)
- U13 pad 9: unconnected-(U13-2Z-Pad9) -> Net-(RN5-R3)
- U14 pad 2: unconnected-(U14-Pad2) -> /Counter/SRV_CLK_TTL
- U15 pad 1: unconnected-(U15-1A-Pad1) -> /Counter/BIT10_TTL
- U15 pad 10: unconnected-(U15-D-Pad10) -> Net-(U13-1C)
- U15 pad 12: unconnected-(U15-1Z-Pad12) -> Net-(RN6-R3)
- U15 pad 13: unconnected-(U15-1Y-Pad13) -> Net-(RN6-R4)
- U15 pad 2: unconnected-(U15-1B-Pad2) -> /Counter/BIT10_TTL
- U15 pad 3: unconnected-(U15-1C-Pad3) -> Net-(U13-1C)
- U15 pad 4: unconnected-(U15-2C-Pad4) -> Net-(U13-1C)
- U15 pad 5: unconnected-(U15-2A-Pad5) -> Net-(U15-2A)
- U15 pad 6: unconnected-(U15-2B-Pad6) -> Net-(U15-2A)
- U15 pad 8: unconnected-(U15-2Y-Pad8) -> Net-(RN6-R1)
- U15 pad 9: unconnected-(U15-2Z-Pad9) -> Net-(RN6-R2)
- U16 pad 1: unconnected-(U16-1A-Pad1) -> Net-(U13-1C)
- U16 pad 10: unconnected-(U16-D-Pad10) -> Net-(U13-1C)
- U16 pad 12: unconnected-(U16-1Z-Pad12) -> Net-(RN7-R3)
- U16 pad 13: unconnected-(U16-1Y-Pad13) -> Net-(RN7-R4)
- U16 pad 2: unconnected-(U16-1B-Pad2) -> Net-(U16-1B)
- U16 pad 3: unconnected-(U16-1C-Pad3) -> Net-(U16-1B)
- U16 pad 4: unconnected-(U16-2C-Pad4) -> Net-(U13-1C)
- U16 pad 5: unconnected-(U16-2A-Pad5) -> Net-(U16-2A)
- U16 pad 6: unconnected-(U16-2B-Pad6) -> Net-(U16-2A)
- U16 pad 8: unconnected-(U16-2Y-Pad8) -> Net-(RN7-R2)
- U16 pad 9: unconnected-(U16-2Z-Pad9) -> Net-(RN7-R1)
- U17 pad 10: unconnected-(U17-D-Pad10) -> Net-(U13-1C)
- U17 pad 12: unconnected-(U17-1Z-Pad12) -> Net-(RN8-R3)
- U17 pad 13: unconnected-(U17-1Y-Pad13) -> Net-(RN8-R4)
- U17 pad 2: unconnected-(U17-1B-Pad2) -> Net-(U13-1C)
- U17 pad 3: unconnected-(U17-1C-Pad3) -> Net-(U13-1C)
- U17 pad 4: unconnected-(U17-2C-Pad4) -> Net-(U13-1C)
- U17 pad 5: unconnected-(U17-2A-Pad5) -> Net-(U13-1C)
- U17 pad 8: unconnected-(U17-2Y-Pad8) -> Net-(RN8-R1)
- U17 pad 9: unconnected-(U17-2Z-Pad9) -> Net-(RN8-R2)
- U18 pad 10: unconnected-(U18-D-Pad10) -> Net-(U13-1C)
- U18 pad 12: unconnected-(U18-1Z-Pad12) -> Net-(RN9-R3)
- U18 pad 13: unconnected-(U18-1Y-Pad13) -> Net-(RN9-R4)
- U18 pad 2: unconnected-(U18-1B-Pad2) -> Net-(U13-1C)
- U18 pad 3: unconnected-(U18-1C-Pad3) -> Net-(U13-1C)
- U18 pad 4: unconnected-(U18-2C-Pad4) -> Net-(U13-1C)
- U18 pad 5: unconnected-(U18-2A-Pad5) -> Net-(U13-1C)
- U18 pad 8: unconnected-(U18-2Y-Pad8) -> Net-(RN9-R2)
- U18 pad 9: unconnected-(U18-2Z-Pad9) -> Net-(RN9-R1)
- U19 pad 1: unconnected-(U19-1A-Pad1) -> GND
- U19 pad 10: unconnected-(U19-D-Pad10) -> GND
- U19 pad 2: unconnected-(U19-1B-Pad2) -> GND
- U19 pad 3: unconnected-(U19-1C-Pad3) -> GND
- U19 pad 4: unconnected-(U19-2C-Pad4) -> Net-(U13-1C)
- U19 pad 5: unconnected-(U19-2A-Pad5) -> Net-(U19-2A)
- U19 pad 6: unconnected-(U19-2B-Pad6) -> Net-(U19-2A)
- U19 pad 8: unconnected-(U19-2Y-Pad8) -> Net-(RN10-R3)
- U19 pad 9: unconnected-(U19-2Z-Pad9) -> Net-(RN10-R4)
- U2 pad 1: Net-(U2-B) -> Net-(U2-A)
- U3 pad 10: Net-(U3-C) -> /Counter/UNIT_SELECT_TTL
- U3 pad 13: unconnected-(U3-~{BO}-Pad13) -> Net-(U11-DOWN)
- U3 pad 15: Net-(U3-A) -> /Counter/CLK_UP
- U4 pad 1: Net-(U3-A) -> /Counter/CLK_UP
- U4 pad 10: unconnected-(U4-C-Pad10) -> /Counter/CLK_UP
- U4 pad 11: Net-(U4-~{LOAD}) -> /Counter/LOAD_TTL______
- U4 pad 13: unconnected-(U4-~{BO}-Pad13) -> Net-(U4-~{BO})
- U4 pad 15: unconnected-(U4-A-Pad15) -> /Counter/CLK_UP
- U4 pad 9: unconnected-(U4-D-Pad9) -> /Counter/CLK_UP
- U5 pad 11: Net-(U4-~{LOAD}) -> /Counter/LOAD_TTL______
- U5 pad 13: Net-(U11-DOWN) -> unconnected-(U5-~{BO}-Pad13)
- U5 pad 3: unconnected-(U5-QA-Pad3) -> /Counter/BIT10_TTL
- U5 pad 4: unconnected-(U5-DOWN-Pad4) -> Net-(U4-~{BO})
- U6 pad 5: Net-(U3-C) -> /Counter/UNIT_SELECT_TTL
- U6 pad 6: Net-(U2-B) -> Net-(U2-A)
- U7 pad 9: unconnected-(U7-Pad9) -> /Counter/UNIT_SELECT_TTL
- U9 pad 11: unconnected-(U9-2B-Pad11) -> Net-(U9-2B)
- U9 pad 12: unconnected-(U9-2A-Pad12) -> Net-(U9-2A)
- U9 pad 4: unconnected-(U9-1Y-Pad4) -> /Counter/LOAD_TTL______
- U9 pad 9: unconnected-(U9-2Y-Pad9) -> /Counter/SRV_CLK_TTL
- X4 pad 1: unconnected-(X4-Pin_1-Pad1) -> /TAG1
- X4 pad 10: unconnected-(X4-Pin_10-Pad10) -> /Bit6
- X4 pad 11: unconnected-(X4-Pin_11-Pad11) -> /Bit7
- X4 pad 12: unconnected-(X4-Pin_12-Pad12) -> /Bit8
- X4 pad 13: unconnected-(X4-Pin_13-Pad13) -> /Bit9
- X4 pad 14: unconnected-(X4-Pin_14-Pad14) -> /Open-Cable-Detect
- X4 pad 15: unconnected-(X4-Pin_15-Pad15) -> /Fault
- X4 pad 16: unconnected-(X4-Pin_16-Pad16) -> /Seek-Error
- X4 pad 17: unconnected-(X4-Pin_17-Pad17) -> /On-Cylinder
- X4 pad 18: unconnected-(X4-Pin_18-Pad18) -> /Index
- X4 pad 19: unconnected-(X4-Pin_19-Pad19) -> /Unit-Ready
- X4 pad 2: unconnected-(X4-Pin_2-Pad2) -> /TAG2
- X4 pad 20: unconnected-(X4-Pin_20-Pad20) -> /Address-Mark-Found
- X4 pad 21: unconnected-(X4-Pin_21-Pad21) -> /Busy
- X4 pad 22: unconnected-(X4-Pin_22-Pad22) -> /Unit-Select-Tag
- X4 pad 23: unconnected-(X4-Pin_23-Pad23) -> /Unit-Select-Bit0
- X4 pad 24: unconnected-(X4-Pin_24-Pad24) -> /Unit-Select-Bit1
- X4 pad 25: unconnected-(X4-Pin_25-Pad25) -> /Sector
- X4 pad 26: unconnected-(X4-Pin_26-Pad26) -> /Unit-Select-Bit2
- X4 pad 27: unconnected-(X4-Pin_27-Pad27) -> /Unit-Select-Bit3
- X4 pad 28: unconnected-(X4-Pin_28-Pad28) -> /Write-Protected
- X4 pad 29: unconnected-(X4-Pin_29-Pad29) -> /Power-Sequence-Hold
- X4 pad 3: unconnected-(X4-Pin_3-Pad3) -> /TAG3
- X4 pad 30: unconnected-(X4-Pin_30-Pad30) -> /Bit10
- X4 pad 31: unconnected-(X4-Pin_31-Pad31) -> //Tag1
- X4 pad 32: unconnected-(X4-Pin_32-Pad32) -> //Tag2
- X4 pad 33: unconnected-(X4-Pin_33-Pad33) -> //Tag3
- X4 pad 34: unconnected-(X4-Pin_34-Pad34) -> //Bit0
- X4 pad 35: unconnected-(X4-Pin_35-Pad35) -> //Bit1
- X4 pad 36: unconnected-(X4-Pin_36-Pad36) -> //Bit2
- X4 pad 37: unconnected-(X4-Pin_37-Pad37) -> //Bit3
- X4 pad 38: unconnected-(X4-Pin_38-Pad38) -> //Bit4
- X4 pad 39: unconnected-(X4-Pin_39-Pad39) -> //Bit5
- X4 pad 4: unconnected-(X4-Pin_4-Pad4) -> /Bit0
- X4 pad 40: unconnected-(X4-Pin_40-Pad40) -> //Bit6
- X4 pad 41: unconnected-(X4-Pin_41-Pad41) -> //Bit7
- X4 pad 42: unconnected-(X4-Pin_42-Pad42) -> //Bit8
- X4 pad 43: unconnected-(X4-Pin_43-Pad43) -> //Bit9
- X4 pad 44: unconnected-(X4-Pin_44-Pad44) -> //Open-Cable-Detect
- X4 pad 45: unconnected-(X4-Pin_45-Pad45) -> //Fault
- X4 pad 46: unconnected-(X4-Pin_46-Pad46) -> //Seek-Error
- X4 pad 47: unconnected-(X4-Pin_47-Pad47) -> //On-Cylinder
- X4 pad 48: unconnected-(X4-Pin_48-Pad48) -> //Index
- X4 pad 49: unconnected-(X4-Pin_49-Pad49) -> //Unit-Ready
- X4 pad 5: unconnected-(X4-Pin_5-Pad5) -> /Bit1
- X4 pad 50: unconnected-(X4-Pin_50-Pad50) -> //Address-Mark-Found
- X4 pad 51: unconnected-(X4-Pin_51-Pad51) -> //Busy
- X4 pad 52: unconnected-(X4-Pin_52-Pad52) -> //Unit-Select-Tag
- X4 pad 53: unconnected-(X4-Pin_53-Pad53) -> //Unit-Select-Bit0
- X4 pad 54: unconnected-(X4-Pin_54-Pad54) -> //Unit-Select-Bit1
- X4 pad 55: unconnected-(X4-Pin_55-Pad55) -> //Sector
- X4 pad 56: unconnected-(X4-Pin_56-Pad56) -> //Unit-Select-Bit2
- X4 pad 57: unconnected-(X4-Pin_57-Pad57) -> //Unit-Select-Bit3
- X4 pad 58: unconnected-(X4-Pin_58-Pad58) -> //Write-Protected
- X4 pad 59: unconnected-(X4-Pin_59-Pad59) -> /Power-Sequence-Pick
- X4 pad 6: unconnected-(X4-Pin_6-Pad6) -> /Bit2
- X4 pad 60: unconnected-(X4-Pin_60-Pad60) -> //Bit10
- X4 pad 7: unconnected-(X4-Pin_7-Pad7) -> /Bit3
- X4 pad 8: unconnected-(X4-Pin_8-Pad8) -> /Bit4
- X4 pad 9: unconnected-(X4-Pin_9-Pad9) -> /Bit5
